File: kicad/caltreat_pcb/caltreat_pcb.kicad_pcb (KiCad board)
At the start: 2 copper layers, 67 x 47 mm, 43 parts, among them J1 Conn_01x12_Pin, J10 Conn_01x02_Pin, J11 Conn_01x02_Pin, J12 Conn_01x02_Pin, J13 Conn_01x02_Pin, J14 Conn_01x02_Pin, J15 Conn_01x02_Pin, J2 Conn_01x12_Pin, J3 Conn_01x02_Pin, J4 Conn_01x02_Pin, J5 Conn_01x02_Pin, J6 Conn_01x02_Pin, J7 Conn_01x02_Pin, J8 Conn_01x02_Pin, J9 Conn_01x02_Pin, Q1 AO3400A, Q2 AO3400A, Q3 AO3400A, Q4 AO3400A, Q5 AO3400A, Q6 AO3400A, Q7 AO3400A, Q8 AO3400A

Commit message: Add level crossing signal firmware
Parts:
- added D1: SK34A-LTP, Diode_SMD:D_SMA, B.Cu at (43.0, 72.0)
- added D2: SK34A-LTP, Diode_SMD:D_SMA, B.Cu at (52.0, 72.0)
- added D3: SK34A-LTP, Diode_SMD:D_SMA, B.Cu at (61.0, 72.0)
- added D4: SK34A-LTP, Diode_SMD:D_SMA, B.Cu at (70.0, 72.0)
- added D5: SK34A-LTP, Diode_SMD:D_SMA, B.Cu at (79.0, 72.0)
- added D6: SK34A-LTP, Diode_SMD:D_SMA, B.Cu at (88.0, 72.0)
- added D7: SK34A-LTP, Diode_SMD:D_SMA, B.Cu at (92.0, 66.0)
- added D8: SK34A-LTP, Diode_SMD:D_SMA, B.Cu at (92.0, 57.0)
Routing:
- net GND: track 59.7 -> 125.5 mm
- net +12V: track 112.0 -> 132.8 mm
- net /FET_DRAIN_CH5: track 14.6 -> 17.7 mm
- net /FET_DRAIN_CH1: track 13.8 -> 16.8 mm
- net /FET_DRAIN_CH4: track 12.8 -> 14.7 mm
- net /FET_DRAIN_CH8: track 18.4 -> 16.9 mm
- net /FET_GATE_CH6: track 7.45 -> 6.01 mm
- net /FET_DRAIN_CH6: track 21.2 -> 22.5 mm
- net /FET_DRAIN_CH7: track 19.2 -> 18.1 mm
- net /FET_GATE_CH7: track 6.45 -> 5.84 mm
Other:
- board text added: "TOOT TOOT"
